File: electronics/pideck.kicad_pcb (KiCad board)
At the start: 2 copper layers, 12 parts, among them IC1 UM6K34NTCN, J1 Conn_01x20_Socket, J2 Conn_01x20_Socket, J3 BM20B_0.8_-34DS-0.4V_53_

Commit message: schematics complete
Parts:
- removed IC1: UM6K34NTCN, UM6K34NTCN:TRANS_UM6J1_ROM
- added Q1: RE1C002UNTCL, RE1C002UNTCL:DIO_RB558WMF_ROM, F.Cu at (105.8, 112.0)
- added Q2: RE1C002UNTCL, RE1C002UNTCL:DIO_RB558WMF_ROM, F.Cu at (112.3, 112.0)
- added Q3: RE1C002UNTCL, RE1C002UNTCL:DIO_RB558WMF_ROM, F.Cu at (105.8, 115.5)
- added Q4: RE1C002UNTCL, RE1C002UNTCL:DIO_RB558WMF_ROM, F.Cu at (112.3, 115.5)
- added Q5: RE1C002UNTCL, RE1C002UNTCL:DIO_RB558WMF_ROM, F.Cu at (105.8, 119.0)
- added Q6: RE1C002UNTCL, RE1C002UNTCL:DIO_RB558WMF_ROM, F.Cu at (112.3, 119.0)
- added Q7: RE1C002UNTCL, RE1C002UNTCL:DIO_RB558WMF_ROM, F.Cu at (105.8, 122.5)
- added Q8: RE1C002UNTCL, RE1C002UNTCL:DIO_RB558WMF_ROM, F.Cu at (112.3, 122.5)
- added R10: 10K, Resistor_SMD:R_0201_0603Metric_Pad0.64x0.40mm_HandSolder, F.Cu at (107.8, 115.5)
- added R11: 10K, Resistor_SMD:R_0201_0603Metric_Pad0.64x0.40mm_HandSolder, F.Cu at (114.3, 115.5)
- added R12: 10K, Resistor_SMD:R_0201_0603Metric_Pad0.64x0.40mm_HandSolder, F.Cu at (110.3, 115.4)
- added R13: 10K, Resistor_SMD:R_0201_0603Metric_Pad0.64x0.40mm_HandSolder, F.Cu at (103.8, 119.0)
- added R14: 10K, Resistor_SMD:R_0201_0603Metric_Pad0.64x0.40mm_HandSolder, F.Cu at (107.8, 119.0)
- added R15: 10K, Resistor_SMD:R_0201_0603Metric_Pad0.64x0.40mm_HandSolder, F.Cu at (114.3, 119.0)
- added R16: 10K, Resistor_SMD:R_0201_0603Metric_Pad0.64x0.40mm_HandSolder, F.Cu at (110.3, 119.0)
- added R17: 10K, Resistor_SMD:R_0201_0603Metric_Pad0.64x0.40mm_HandSolder, F.Cu at (103.8, 122.5)
- added R18: 10K, Resistor_SMD:R_0201_0603Metric_Pad0.64x0.40mm_HandSolder, F.Cu at (107.8, 122.5)
- added R19: 10K, Resistor_SMD:R_0201_0603Metric_Pad0.64x0.40mm_HandSolder, F.Cu at (114.3, 122.5)
- added R20: 10K, Resistor_SMD:R_0201_0603Metric_Pad0.64x0.40mm_HandSolder, F.Cu at (110.3, 122.5)
- added R5: 10K, Resistor_SMD:R_0201_0603Metric_Pad0.64x0.40mm_HandSolder, F.Cu at (103.8, 112.0)
- added R6: 10K, Resistor_SMD:R_0201_0603Metric_Pad0.64x0.40mm_HandSolder, F.Cu at (107.8, 112.0)
- added R7: 10K, Resistor_SMD:R_0201_0603Metric_Pad0.64x0.40mm_HandSolder, F.Cu at (114.3, 112.0)
- added R8: 10K, Resistor_SMD:R_0201_0603Metric_Pad0.64x0.40mm_HandSolder, F.Cu at (110.3, 112.0)
- added R9: 10K, Resistor_SMD:R_0201_0603Metric_Pad0.64x0.40mm_HandSolder, F.Cu at (103.8, 115.4)
- moved R4 60.3 mm to (113.0, 132.0)
- moved R3 59.6 mm to (105.4, 131.6)
- moved R1 55.9 mm to (105.8, 127.4)
- moved R2 55.7 mm to (112.4, 126.6)
- moved C1 35.7 mm to (107.3, 105.8)
- moved C3 35.3 mm to (110.3, 104.0)
- moved LDO1 34.4 mm to (110.3, 106.8)
- moved C2 30.7 mm to (107.3, 107.8), turned to 180 degrees
- moved J3 2.70 mm to (108.5, 140.2)
Connections:
- net GP10 renamed ROW5
- net GP11 renamed ROW4
- net GP12 renamed ROW3
- net GP13 renamed ROW2
- net GP14 renamed ROW1
- net GP8 renamed ROW7
- net GP9 renamed ROW6
- C2 pad 1: +3V3 -> KB_BLK_LED_A
- J1 pad 10: unconnected-(J1-Pin_10-Pad10) -> PANNEL_BLK_LED_K_3V3
- J1 pad 9: unconnected-(J1-Pin_9-Pad9) -> KB_BLK_LED_K_3V3
- J2 pad 5: +3V3 -> KB_BLK_LED_A
- J3 pad 17: unconnected-(J3-Pad17) -> KB_BLK_LED_A
- J3 pad 18: unconnected-(J3-Pad18) -> TP_MOTION_1V8
- J3 pad 19: unconnected-(J3-Pad19) -> KB_BLK_LED_A
- J3 pad 20: unconnected-(J3-Pad20) -> TP_SHUTDOWN_1V8
- J3 pad 21: unconnected-(J3-Pad21) -> KB_BLK_LED_K_1V8
- J3 pad 28: unconnected-(J3-Pad28) -> TP_BLK_LED_K_1V8
- J3 pad 29: unconnected-(J3-Pad29) -> PANNEL_BLK_LED_K_1V8
- J3 pad 32: unconnected-(J3-Pad32) -> TP_RESET_1V8
- LDO1 pad 3: +3V3 -> KB_BLK_LED_A
- LDO1 pad 4: +3V3 -> KB_BLK_LED_A
- LDO1 pad 5: +3V3 -> KB_BLK_LED_A
- R3 pad 2: +3V3 -> KB_BLK_LED_A
- R4 pad 2: +3V3 -> KB_BLK_LED_A

Commit message: routed
Parts:
- moved R2 20.7 mm to (104.2, 145.6), turned to 90 degrees
- moved R1 18.2 mm to (106.2, 145.6), turned to 90 degrees
- moved R17 14.8 mm to (114.2, 112.0), turned to 90 degrees
- moved R5 13.2 mm to (114.2, 120.0), turned to 90 degrees
- moved Q7 12.3 mm to (112.2, 112.0), turned to 90 degrees
- moved Q2 12.0 mm to (112.2, 124.0)
- moved R7 12.0 mm to (114.2, 124.0)
- moved R8 12.0 mm to (110.2, 124.0), turned to -90 degrees
- moved R15 11.6 mm to (103.8, 124.0), turned to -90 degrees
- moved R18 10.8 mm to (110.2, 112.0), turned to -90 degrees
- moved R11 10.5 mm to (103.8, 116.0), turned to -90 degrees
- moved Q1 10.3 mm to (112.2, 120.0), turned to 90 degrees
- moved R6 8.38 mm to (110.2, 120.0)
- moved Q6 8.21 mm to (105.8, 124.0), turned to -90 degrees
- moved Q4 6.53 mm to (105.8, 116.0), turned to -90 degrees
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Connections:
- J1 pad 13: GND -> unconnected-(J1-GND-Pad13)
- J1 pad 4: unconnected-(J1-GP2-Pad4) -> TP_MOTION_3V3
- J1 pad 5: unconnected-(J1-GP3-Pad5) -> TP_SHUTDOWN_3V3
- J1 pad 6: unconnected-(J1-GP4-Pad6) -> TP_RESET_3V3
- J1 pad 7: unconnected-(J1-GP5-Pad7) -> TP_BLK_LED_K_3V3
- J1 pad 8: GND -> unconnected-(J1-GND-Pad8)
- J2 pad 13: GND -> unconnected-(J2-GND-Pad13)
- J2 pad 18: GND -> unconnected-(J2-GND-Pad18)
- J2 pad 3: GND -> unconnected-(J2-GND-Pad3)
- J2 pad 8: GND -> unconnected-(J2-GND-Pad8)
Routing:
- net +1V8: track 0.00 -> 122.8 mm, vias 0 -> 2
- net KB_BLK_LED_A: track 0.00 -> 81.2 mm, vias 0 -> 2
- net TP_SCL_1V8: track 0.00 -> 58.2 mm, vias 0 -> 2
- net +2V8: track 0.00 -> 55.6 mm, vias 0 -> 2
- net TP_SDA_1V8: track 0.00 -> 53.3 mm, vias 0 -> 2
- net KB_BLK_LED_K_1V8: track 0.00 -> 41.6 mm, vias 0 -> 2
- net PANNEL_BLK_LED_K_1V8: track 0.00 -> 39.8 mm, vias 0 -> 2
- net GND: track 0.00 -> 37.8 mm, vias 0 -> 2
- net TP_SCL_3V3: track 0.00 -> 37.7 mm, vias 0 -> 3
- net TP_MOTION_1V8: track 0.00 -> 34.2 mm, vias 0 -> 2
- net TP_SDA_3V3: track 0.00 -> 32.7 mm, vias 0 -> 3
- net TP_RESET_1V8: track 0.00 -> 32.0 mm, vias 0 -> 2
- net TP_SHUTDOWN_1V8: track 0.00 -> 31.6 mm, vias 0 -> 2
- net TP_BLK_LED_K_3V3: track 0.00 -> 31.3 mm, vias 0 -> 1
- net TP_RESET_3V3: track 0.00 -> 25.5 mm, vias 0 -> 1
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Other:
- board outline added: 21.3 x 52 mm
