File: electronics/pideck.kicad_pcb (KiCad board)
At the start: 2 copper layers, 21.3 x 52 mm, 35 parts, among them J1 Conn_01x20_Socket, J2 Conn_01x20_Socket, J3 BM20B_0.8_-34DS-0.4V_53_, Q1 RE1C002UNTCL, Q2 RE1C002UNTCL, Q3 RE1C002UNTCL, Q4 RE1C002UNTCL, Q5 RE1C002UNTCL, Q6 RE1C002UNTCL, Q7 RE1C002UNTCL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

Commit message: new routing
Parts:
- moved R2 51.2 mm to (137.9, 107.0)
- moved R1 49.0 mm to (136.4, 107.0)
- moved R15 46.6 mm to (137.8, 92.3), turned to 180 degrees
- moved R13 46.5 mm to (137.8, 88.4), turned to 180 degrees
- moved Q6 46.5 mm to (140.4, 93.0)
- moved Q5 46.5 mm to (140.4, 89.1)
- moved R16 42.9 mm to (137.8, 93.5), turned to 0 degrees
- moved R14 42.8 mm to (137.8, 89.5), turned to 0 degrees
- moved C2 41.9 mm to (137.2, 78.4), turned to 90 degrees
- moved R11 39.6 mm to (133.2, 89.5), turned to 0 degrees
- moved C1 38.4 mm to (134.2, 78.4), turned to -90 degrees
- moved R12 37.6 mm to (133.2, 88.4), turned to 180 degrees
- moved Q4 36.7 mm to (130.7, 89.1), turned to 90 degrees
- moved J1 36.2 mm to (144.5, 75.8)
- moved C3 36.1 mm to (135.7, 78.4), turned to -90 degrees
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Connections:
- J1 pad 3: GND -> unconnected-(J1-GND-Pad3)
- J2 pad 3: unconnected-(J2-GND-Pad3) -> GND
Routing:
- net TP_SCL_1V8: track 58.2 -> 29.0 mm, vias 2 -> 3
- net TP_BLK_LED_K_3V3: track 31.3 -> 7.70 mm, vias 1 -> 0
- net TP_SDA_1V8: track 53.3 -> 34.0 mm, vias 2 -> 3
- net TP_BLK_LED_K_1V8: track 25.0 -> 43.9 mm
- net TP_RESET_3V3: track 25.5 -> 7.12 mm, vias 1 -> 0
- net TP_RESET_1V8: track 32.0 -> 48.4 mm
- net TP_SCL_3V3: track 37.7 -> 21.4 mm, vias 3 -> 2
- net TP_MOTION_3V3: track 16.8 -> 30.3 mm
- net KB_BLK_LED_K_3V3: track 19.1 -> 7.22 mm, vias 1 -> 0
- net +2V8: track 55.6 -> 66.8 mm
- net +1V8: track 122.8 -> 133.5 mm, vias 2 -> 11
- net PANNEL_BLK_LED_K_3V3: track 17.0 -> 7.79 mm, vias 1 -> 0
- net PANNEL_BLK_LED_K_1V8: track 39.8 -> 30.8 mm
- net KB_BLK_LED_K_1V8: track 41.6 -> 33.0 mm
- net TP_SHUTDOWN_1V8: track 31.6 -> 39.8 mm
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- added copper zone on B.Cu, net GND
- added copper zone on F.Cu, net GND
