File: electronics/pideck.kicad_sch (KiCad schematic)
At the start: 12 parts, among them IC1 UM6K34NTCN, J1 Conn_01x20_Socket, J2 Conn_01x20_Socket, J3 BM20B_0.8_-34DS-0.4V_53_

Commit message: schematics complete
Parts:
- removed IC1: UM6K34NTCN, UM6K34NTCN:TRANS_UM6J1_ROM, symbol UM6K34NTCN:UM6K34NTCN
- removed R1, R2, R3, R4: 10k, Resistor_SMD:R_0201_0603Metric_Pad0.64x0.40mm_HandSolder, symbol Device:R_Small
- added Q7, Q8: RE1C002UNTCL, RE1C002UNTCL:DIO_RB558WMF_ROM, symbol RE1C002UNTCL:RE1C002UNTCL
- added R17, R18, R19, R20: 10K, Resistor_SMD:R_0201_0603Metric_Pad0.64x0.40mm_HandSolder, symbol Device:R_Small
Connections:
- net +1V8: now also Q7.1 (G), Q8.1 (G), R17.1, R19.1
- net +3V3: now also J3.17, J3.19, R18.1, R20.1
- net PANNEL_BLK_LED_K_3V3: now reaches J1.10 (GP7)
- net PANNEL_BLK_LED_K_3V3: now also Q8.3 (D), R20.2
- net KB_BLK_LED_K_3V3: now reaches J1.9 (GP6)
- net KB_BLK_LED_K_3V3: now also Q7.3 (D), R18.2
- net TP_MOTION_1V8: now reaches J3.18
- net TP_SHUTDOWN_1V8: now reaches J3.20
- net KB_BLK_LED_K_1V8: now reaches J3.21
- net KB_BLK_LED_K_1V8: now also Q7.2 (S), R17.2
- net TP_BLK_LED_K_1V8: now reaches J3.28
- net PANNEL_BLK_LED_K_1V8: now reaches J3.29
- net PANNEL_BLK_LED_K_1V8: now also Q8.2 (S), R19.2
- net TP_RESET_1V8: now reaches J3.32
- net GP10 renamed ROW5
- net GP11 renamed ROW4
- net GP12 renamed ROW3
- net GP13 renamed ROW2
- net GP14 renamed ROW1
- net GP8 renamed ROW7
- net GP9 renamed ROW6
Other:
- added sheet Track Pad (untitled.kicad_sch)
- note added: "9900 KEYBOARD"
- note removed: "9900 TRACKPAD"
- note removed: "TRACK PAD"
- moved on the sheet: C1, C2, C3, J3, LDO1

Commit message: routed
Connections:
- net GND: no longer J1.13 (GND), J1.8 (GND), J2.13 (GND), J2.18 (GND), J2.3 (GND), J2.8 (GND)
- net TP_MOTION_3V3: now reaches J1.4 (GP2)
- net TP_SHUTDOWN_3V3: now reaches J1.5 (GP3)
- net TP_RESET_3V3: now reaches J1.6 (GP4)
- net TP_BLK_LED_K_3V3: now reaches J1.7 (GP5)
- no-connect marks 5 -> 15

Commit message: new routing
Connections:
- net GND: now also J2.3 (GND); no longer J1.3 (GND)
Changed lines of the file:
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@@
 	(wire
 		(pts
+			(xy 83.82 135.89) (xy 86.36 135.89)
+		)
+		(stroke
+			(width 0)
+			(type default)
+		)
+	)
+	(wire
+		(pts
 			(xy 175.26 46.99) (xy 179.07 46.99)
 		)
@@
 	(symbol
 		(lib_id "power:GND")
-		(at 50.8 135.89 270)
+		(at 176.53 72.39 270)
 		(unit 1)
 		(exclude_from_sim no)
@@
 		(on_board yes)
 		(dnp no)
-		(fields_autoplaced yes)
-		(property "Reference" "#PWR04"
-			(at 44.45 135.89 0)
+		(property "Reference" "#PWR014"
+			(at 170.18 72.39 0)
 			(effects
 				(font
@@
 		)
 		(property "Value" "GND"
-			(at 46.99 135.8899 90)
+			(at 172.72 72.39 90)
 			(effects
 				(font
@@
 		)
 		(property "Footprint" ""
-			(at 50.8 135.89 0)
+			(at 176.53 72.39 0)
 			(effects
 				(font
@@
 		)
 		(property "Datasheet" ""
-			(at 50.8 135.89 0)
+			(at 176.53 72.39 0)
 			(effects
 				(font
@@
 		)
 		(property "Description" "Power symbol creates a global label with name \"GND\" , ground"
-			(at 50.8 135.89 0)
+			(at 176.53 72.39 0)
 			(effects
 				(font
@@
 			(project "pideck"
 				(path "/731f0414-be38-4c27-b718-5d8edfd5df05"
-					(reference "#PWR04")
+					(reference "#PWR014")
 					(unit 1)
 				)
@@
 	)
 	(symbol
-		(lib_id "power:GND")
-		(at 176.53 72.39 270)
+		(lib_id "power:+3V3")
+		(at 166.37 77.47 270)
 		(unit 1)
 		(exclude_from_sim no)
@@
 		(on_board yes)
 		(dnp no)
-		(property "Reference" "#PWR014"
-			(at 170.18 72.39 0)
+		(fields_autoplaced yes)
+		(property "Reference" "#PWR011"
+			(at 162.56 77.47 0)
 			(effects
 				(font
@@
 			)
 		)
-		(property "Value" "GND"
-			(at 172.72 72.39 90)
+		(property "Value" "+3V3"
+			(at 170.18 77.4699 90)
 			(effects
 				(font
 					(size 1.27 1.27)
 				)
-				(justify right)
+				(justify left)
 			)
 		)
 		(property "Footprint" ""
-			(at 176.53 72.39 0)
+			(at 166.37 77.47 0)
 			(effects
 				(font
@@
 		)
 		(property "Datasheet" ""
-			(at 176.53 72.39 0)
+			(at 166.37 77.47 0)
 			(effects
 				(font
@@
 			)
 		)
-		(property "Description" "Power symbol creates a global label with name \"GND\" , ground"
-			(at 176.53 72.39 0)
+		(property "Description" "Power symbol creates a global label with name \"+3V3\""
+			(at 166.37 77.47 0)
 			(effects
 				(font
@@
 			(project "pideck"
 				(path "/731f0414-be38-4c27-b718-5d8edfd5df05"
-					(reference "#PWR014")
+					(reference "#PWR011")
 					(unit 1)
 				)
@@
 	)
 	(symbol
-		(lib_id "power:+3V3")
-		(at 166.37 77.47 270)
+		(lib_id "power:GND")
+		(at 86.36 135.89 90)
 		(unit 1)
 		(exclude_from_sim no)
@@
 		(dnp no)
 		(fields_autoplaced yes)
-		(property "Reference" "#PWR011"
-			(at 162.56 77.47 0)
+		(property "Reference" "#PWR05"
+			(at 92.71 135.89 0)
 			(effects
 				(font
@@
 			)
 		)
-		(property "Value" "+3V3"
-			(at 170.18 77.4699 90)
+		(property "Value" "GND"
+			(at 90.17 135.8899 90)
 			(effects
 				(font
 					(size 1.27 1.27)
 				)
-				(justify left)
+				(justify right)
 			)
 		)
 		(property "Footprint" ""
-			(at 166.37 77.47 0)
+			(at 86.36 135.89 0)
 			(effects
 				(font
@@
 		)
 		(property "Datasheet" ""
-			(at 166.37 77.47 0)
+			(at 86.36 135.89 0)
 			(effects
 				(font
@@
 			)
 		)
-		(property "Description" "Power symbol creates a global label with name \"+3V3\""
-			(at 166.37 77.47 0)
+		(property "Description" "Power symbol creates a global label with name \"GND\" , ground"
+			(at 86.36 135.89 0)
 			(effects
 				(font
@@
 			(project "pideck"
 				(path "/731f0414-be38-4c27-b718-5d8edfd5df05"
-					(reference "#PWR011")
+					(reference "#PWR05")
 					(unit 1)
 				)
