File: electronics/keyboard_hat/pideck.kicad_sch (KiCad schematic)
At the start: 13 parts, among them J1 Conn_01x20_Socket, J2 Conn_01x20_Socket, J3 BM20B_0.8_-34DS-0.4V_53_, Q7 RE1C002UNTCL, Q8 RE1C002UNTCL

Commit message: finished hat and started full deck
Connections:
- net KB_BLK_LED_K_1V8: now also J3.23, J3.25, J3.27
- no-connect marks 15 -> 12
Changed lines of the file:
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@@
+	)
+	(junction
+		(at 176.53 57.15)
+		(diameter 0)
+		(color 0 0 0 0)
 	)
 	(junction
@@
 	)
 	(junction
+		(at 176.53 59.69)
+		(diameter 0)
+		(color 0 0 0 0)
+	)
+	(junction
 		(at 48.26 66.04)
 		(diameter 0)
@@
 	)
 	(junction
+		(at 176.53 62.23)
+		(diameter 0)
+		(color 0 0 0 0)
+	)
+	(junction
 		(at 85.09 66.04)
 		(diameter 0)
@@
 	)
 	(no_connect
-		(at 179.07 59.69)
-	)
-	(no_connect
-		(at 179.07 64.77)
-	)
-	(no_connect
 		(at 83.82 130.81)
 	)
@@
 	)
 	(no_connect
-		(at 179.07 62.23)
-	)
-	(no_connect
 		(at 83.82 151.13)
 	)
@@
 	(wire
 		(pts
+			(xy 176.53 62.23) (xy 176.53 59.69)
+		)
+		(stroke
+			(width 0)
+			(type default)
+		)
+	)
+	(wire
+		(pts
 			(xy 175.26 39.37) (xy 179.07 39.37)
 		)
@@
 	(wire
 		(pts
+			(xy 176.53 64.77) (xy 176.53 62.23)
+		)
+		(stroke
+			(width 0)
+			(type default)
+		)
+	)
+	(wire
+		(pts
 			(xy 83.82 171.45) (xy 86.36 171.45)
 		)
@@
 	(wire
 		(pts
+			(xy 179.07 64.77) (xy 176.53 64.77)
+		)
+		(stroke
+			(width 0)
+			(type default)
+		)
+	)
+	(wire
+		(pts
 			(xy 83.82 135.89) (xy 86.36 135.89)
 		)
@@
 	(wire
 		(pts
+			(xy 176.53 59.69) (xy 179.07 59.69)
+		)
+		(stroke
+			(width 0)
+			(type default)
+		)
+	)
+	(wire
+		(pts
 			(xy 50.8 143.51) (xy 53.34 143.51)
 		)
@@
 	(wire
 		(pts
+			(xy 179.07 62.23) (xy 176.53 62.23)
+		)
+		(stroke
+			(width 0)
+			(type default)
+		)
+	)
+	(wire
+		(pts
 			(xy 208.28 119.38) (xy 209.55 119.38)
 		)
@@
 	(wire
 		(pts
-			(xy 175.26 57.15) (xy 179.07 57.15)
+			(xy 175.26 57.15) (xy 176.53 57.15)
 		)
 		(stroke
@@
 	(wire
 		(pts
+			(xy 176.53 57.15) (xy 179.07 57.15)
+		)
+		(stroke
+			(width 0)
+			(type default)
+		)
+	)
+	(wire
+		(pts
 			(xy 176.53 31.75) (xy 179.07 31.75)
 		)
@@
 		)
 		(stroke
+			(width 0)
+			(type default)
+		)
+	)
+	(wire
+		(pts
+			(xy 176.53 57.15) (xy 176.53 59.69)
+		)
+		(stroke

Commit message: updated schematic to new chip and completed layout
Parts:
- removed Q7, Q8: RE1C002UNTCL, RE1C002UNTCL:DIO_RB558WMF_ROM, symbol RE1C002UNTCL:RE1C002UNTCL
- removed R17, R18, R19, R20: 10K, Resistor_SMD:R_0201_0603Metric_Pad0.64x0.40mm_HandSolder, symbol Device:R_Small
- added C4, C5: 0.1uF, Capacitor_SMD:C_0603_1608Metric, symbol Device:C
- added R1: 10k, Resistor_SMD:R_0603_1608Metric, symbol Device:R_US
- added U3: TXS0108EPWR, Package_SO:TSSOP-20_4.4x6.5mm_P0.65mm, symbol Logic_LevelTranslator:TXS0108EPW
- C1, C2, C3: footprint Capacitor_SMD:C_0201_0603Metric -> Capacitor_SMD:C_0603_1608Metric
Connections:
- net +1V8: now also C5.2, R1.2, U3.10 (OE), U3.2 (VCCA)
- net +3V3: now also C4.1, U3.19 (VCCB)
- net GND: now also C4.2, C5.1, R1.1, U3.11 (GND)
- net KB_BLK_LED_K_1V8: now also U3.8 (A7)
- net KB_BLK_LED_K_3V3: now also U3.13 (B7)
- net PANNEL_BLK_LED_K_1V8: now also U3.9 (A8)
- net PANNEL_BLK_LED_K_3V3: now also U3.12 (B8)
- net TP_BLK_LED_K_1V8: now also U3.7 (A6)
- net TP_BLK_LED_K_3V3: now also U3.14 (B6)
- net TP_MOTION_1V8: now also U3.4 (A3)
- net TP_MOTION_3V3: now also U3.17 (B3)
- net TP_RESET_1V8: now also U3.6 (A5)
- net TP_RESET_3V3: now also U3.15 (B5)
- net TP_SCL_1V8: now also U3.1 (A1)
- net TP_SCL_3V3: now also U3.20 (B1)
- net TP_SDA_1V8: now also U3.3 (A2)
- net TP_SDA_3V3: now also U3.18 (B2)
- net TP_SHUTDOWN_1V8: now also U3.5 (A4)
- net TP_SHUTDOWN_3V3: now also U3.16 (B4)
Other:
- removed sheet Track Pad
