File: electronics/pideck/pideck.kicad_sch (KiCad schematic)
At the start: 50 parts, among them J1 BM20B_0.8_-34DS-0.4V_53_, Q1 RE1C002UNTCL, Q2 RE1C002UNTCL, Q3 RE1C002UNTCL, Q4 RE1C002UNTCL, Q5 RE1C002UNTCL, Q6 RE1C002UNTCL, Q7 RE1C002UNTCL, Q8 RE1C002UNTCL, U1 RP2040, U2 AP7312-1828W6-7, U3 GD25Q16ETIGR, X1 ABM8-272-T3

Commit message: Adding ethernet, hdmi, and battery to CM5
Parts:
- removed Q1, Q2, Q3, Q4, Q5, Q6, Q7, Q8: RE1C002UNTCL, RE1C002UNTCL:DIO_RB558WMF_ROM, symbol RE1C002UNTCL:RE1C002UNTCL
- removed R10, R11, R12, R13, R14, R15, R16, R17, R18, R4, R5, R8, R9: 10K, Resistor_SMD:R_0201_0603Metric, symbol Device:R_Small
- added BT1: BAT-HLD-001-THM, BAT-HLD-001-THM:BAT_BAT-HLD-001-THM, symbol BAT-HLD-001-THM:BAT-HLD-001-THM
- added C18, C19: 1uF, Capacitor_SMD:C_0603_1608Metric_Pad1.08x0.95mm_HandSolder, symbol Device:C_Small
- added C20, C22, C23: 100nF, Capacitor_SMD:C_0603_1608Metric_Pad1.08x0.95mm_HandSolder, symbol Device:C_Small
- added C21: 10uF, Capacitor_SMD:C_0603_1608Metric_Pad1.08x0.95mm_HandSolder, symbol Device:C_Small
- added J2: ARJM11D7-502-AB-EW2, ARJM11D7-502-AB-EW2:ABRACON_ARJM11D7-502-AB-EW2, symbol ARJM11D7-502-AB-EW2:ARJM11D7-502-AB-EW2
- added J3: HDMI_D_1.4, Connector_Video:HDMI_Micro-D_Molex_46765-1x01, symbol Connector:HDMI_D_1.4
- added J4: Micro_SD_Card_Det2, Connector_Card:microSD_HC_Hirose_DM3AT-SF-PEJM5, symbol Connector:Micro_SD_Card_Det2
- added Module1: ComputeModule5-CM5, CM5IO:Raspberry-Pi-5-Compute-Module, symbol CM5IO:ComputeModule5-CM5
- added U4: RT9742GGJ5, Package_TO_SOT_SMD:SOT-23-5, symbol CM5IO:RT9742GGJ5
- added U5: TXS0108EPW, Package_SO:TSSOP-20_4.4x6.5mm_P0.65mm, symbol Logic_LevelTranslator:TXS0108EPW
- added U6: RT9742SNGV, Package_TO_SOT_SMD:TSOT-23_HandSoldering, symbol CM5IO:RT9742SNGV
- C1, C10, C11, C12, C13, C14, C15, C16, C17, C2, C3, C4, C5, C6, C7, C8, C9: footprint Capacitor_SMD:C_0201_0603Metric -> Capacitor_SMD:C_0603_1608Metric_Pad1.08x0.95mm_HandSolder
- R1, R2, R3: footprint Resistor_SMD:R_0201_0603Metric -> Resistor_SMD:R_0603_1608Metric_Pad0.98x0.95mm_HandSolder
- R4: renamed from R20; footprint Resistor_SMD:R_0201_0603Metric -> Resistor_SMD:R_0603_1608Metric_Pad0.98x0.95mm_HandSolder
- R5: renamed from R19; footprint Resistor_SMD:R_0201_0603Metric -> Resistor_SMD:R_0603_1608Metric_Pad0.98x0.95mm_HandSolder
- R6, R7: value 10K -> 470; footprint Resistor_SMD:R_0201_0603Metric -> Resistor_SMD:R_0603_1608Metric_Pad0.98x0.95mm_HandSolder
Connections:
- net +1V8: now also R3.2, C19.2, U5.10 (OE), U5.2 (VCCA); no longer R7.1
- net +3V3: now also C18.1, U4.5 (IN), U5.19 (VCCB); no longer R3.1, R6.1
- net GND: now also R3.1, C18.2, C19.1, C20.2, C21.2, C22.2, C23.2, J2.S1 (SHIELD), J2.S2 (SHIELD__1), J3.10 (D0S), J3.13 (CKS), J3.16 (GND), J3.4 (D2S), J3.7 (D1S), J3.SH, J4.11 (SHIELD), J4.6 (VSS), U4.2 (GND), U5.11 (GND), U6.3 (GND)
- net KB_BLK_LED_K_1V8: now also U5.1 (A1)
- net KB_BLK_LED_K_3V3: now also U5.20 (B1); no longer R3.2
- net PANNEL_BLK_LED_K_1V8: now also U5.3 (A2)
- net PANNEL_BLK_LED_K_3V3: now also U5.18 (B2); no longer R6.2
- net TP_BLK_LED_K_1V8: now also U5.6 (A5); no longer R7.2
- net TP_BLK_LED_K_3V3: now also U5.15 (B5)
- net TP_MOTION_1V8: now also U5.4 (A3)
- net TP_MOTION_3V3: now also U5.17 (B3)
- net TP_RESET_1V8: now also U5.5 (A4)
- net TP_RESET_3V3: now also U5.16 (B4)
- net TP_SCL_1V8: now also U5.8 (A7)
- net TP_SCL_3V3: now also U5.13 (B7)
- net TP_SDA_1V8: now also U5.9 (A8)
- net TP_SDA_3V3: now also U5.12 (B8)
- net TP_SHUTDOWN_1V8: now also U5.7 (A6)
- net TP_SHUTDOWN_3V3: now also U5.14 (B6)
- new net: BT1.N, Module1.74 (GND)
- new net: BT1.P1, BT1.P2, BT1.P3, BT1.P4, Module1.76 (VBAT)
- new net: C20.1, J2.P5 (CT_1), J2.P6 (CT_2)
- new net: J2.P12, R6.2
- new net: J2.P14, R7.2
- new net +3v3: J2.P11, J2.P13
- new net +5V: C23.1, U6.1 (IN)
- new net ETH_LEDG: Module1.17 (Ethernet_nLED2(3.3v)), R6.1
- new net ETH_LEDY: Module1.15 (Ethernet_nLED3(3.3v)), R7.1
- new net HDMI0_CEC: J3.15 (CEC), Module1.151 (HDMI0_CEC)
- new net HDMI0_CK_N: J3.14 (CK-)
- new net HDMI0_CK_P: J3.12 (CK+)
- new net HDMI0_D0_N: J3.11 (D0-), Module1.184 (HDMI0_TX0_N)
- new net HDMI0_D0_P: J3.9 (D0+), Module1.182 (HDMI0_TX0_P)
- new net HDMI0_D1_N: J3.8 (D1-), Module1.178 (HDMI0_TX1_N)
- new net HDMI0_D1_P: J3.6 (D1+), Module1.176 (HDMI0_TX1_P)
- new net HDMI0_D2_N: J3.5 (D2-), Module1.172 (HDMI0_TX2_N)
- new net HDMI0_D2_P: J3.3 (D2+), Module1.170 (HDMI0_TX2_P)
- new net HDMI0_HOTPLUG: J3.1 (HPD/HEAC-), Module1.153 (HDMI0_HOTPLUG)
- new net HDMI0_SCL: J3.17 (SCL), Module1.200 (HDMI0_SCL)
- new net HDMI0_SDA: J3.18 (SDA), Module1.199 (HDMI0_SDA)
- new net HDMI_5v: C22.1, J3.19 (+5V), U6.2 (OUT)
- new net SD_CLK: Module1.57 (SD_CLK)
- new net SD_CMD: Module1.62 (SD_CMD)
- new net SD_DAT0: J4.7 (DAT0), Module1.63 (SD_DAT0)
- new net SD_DAT1: J4.8 (DAT1), Module1.67 (SD_DAT1)
- new net SD_DAT2: J4.1 (DAT2), Module1.69 (SD_DAT2)
- new net SD_DAT3: J4.2 (DAT3/CD), Module1.61 (SD_DAT3)
- new net SD_PWR: C21.1, J4.4 (VDD), U4.1 (OUT)
- new net SD_PWR_ON: Module1.75 (SD_PWR_ON), U4.4 (EN)
- new net TRD0_N: J2.P2 (TD1-), Module1.12 (Ethernet_Pair0_P)
- new net TRD0_P: J2.P1 (TD1+), Module1.10 (Ethernet_Pair0_N)
- new net TRD1_N: J2.P4 (TD2-), Module1.6 (Ethernet_Pair1_N)
- new net TRD1_P: J2.P3 (TD2+), Module1.4 (Ethernet_Pair1_P)
- new net TRD2_N: J2.P8 (TD3-), Module1.9 (Ethernet_Pair2_N)
- new net TRD2_P: J2.P7 (TD3+), Module1.11 (Ethernet_Pair2_P)
- new net TRD3_N: J2.P10 (TD4-), Module1.3 (Ethernet_Pair3_P)
- new net TRD3_P: J2.P9 (TD4+), Module1.5 (Ethernet_Pair3_N)
- no-connect marks 2 -> 5
Other:
- note added: "Ethernet"
- note added: "SD CARD"

Commit message: added usb
Parts:
- added C24, C25: 0.1uF, Capacitor_SMD:C_0603_1608Metric_Pad1.08x0.95mm_HandSolder, symbol Device:C_Small
- added C26: 120uF, Capacitor_SMD:C_0603_1608Metric_Pad1.08x0.95mm_HandSolder, symbol Device:C_Small
- added C27: 10uF, Capacitor_SMD:C_0603_1608Metric_Pad1.08x0.95mm_HandSolder, symbol Device:C_Small
- added J5, J6: USB_C_Receptacle, Connector_USB:USB_C_Receptacle_Molex_105450-0101, symbol Connector:USB_C_Receptacle
- added R8: 20K, Resistor_SMD:R_0603_1608Metric_Pad0.98x0.95mm_HandSolder, symbol Device:R_Small
- added U7: AP22653W6-7, AP22653W6-7:SOT95P280X145-6N, symbol AP22653W6-7:AP22653W6-7
Connections:
- net USB_D+ is gone; now on net KB_USB_D+: R4.1
- net USB_D- is gone; now on net KB_USB_D-: R5.1
- net +5V: now also C24.1, C27.1, U7.1 (IN)
- net GND: now also C24.2, C25.2, C26.2, C27.2, J5.A1 (GND), J5.A12 (GND), J5.B1 (GND), J5.B12 (GND), J5.S1 (SHIELD), J6.A1 (GND), J6.A12 (GND), J6.B1 (GND), J6.B12 (GND), J6.S1 (SHIELD), R8.2, U7.2 (GND)
- net CC1: now reaches Module1.94 (CC1)
- net CC1: now also J5.A5 (CC1), J6.A5 (CC1)
- net CC2: now reaches Module1.96 (CC2)
- net CC2: now also J5.B5 (CC2), J6.B5 (CC2)
- net KB_USB_D-: now reaches Module1.103 (USB2_N)
- net KB_USB_D+: now reaches Module1.105 (USB2_P)
- net VBUS_EN: now reaches Module1.111 (VBUS_EN)
- net VBUS_EN: now also U7.3 (EN)
- net USB3-0-RX_N: now reaches Module1.128 (USB3-0-RX_N)
- net USB3-0-RX_N: now also J5.A10 (RX2-), J5.B10 (RX1-)
- net USB3-0-RX_P: now reaches Module1.130 (USB3-0-RX_P)
- net USB3-0-RX_P: now also J5.A11 (RX2+), J5.B11 (RX1+)
- net USB3-0-D_P: now reaches Module1.134 (USB3-0-D_P)
- net USB3-0-D_P: now also J5.A6 (D+), J5.B6 (D+)
- net USB3-0-D_N: now reaches Module1.136 (USB3-0-D_N)
- net USB3-0-D_N: now also J5.A7 (D-), J5.B7 (D-)
- net USB3-0-TX_N: now reaches Module1.140 (USB3-0-TX_N)
- net USB3-0-TX_N: now also J5.A3 (TX1-), J5.B3 (TX2-)
- net USB3-0-TX_P: now reaches Module1.142 (USB3-0-TX_P)
- net USB3-0-TX_P: now also J5.A2 (TX1+), J5.B2 (TX2+)
- net USB3-1-RX_N: now reaches Module1.157 (USB3-1-RX_N)
- net USB3-1-RX_N: now also J6.A10 (RX2-), J6.B10 (RX1-)
- net USB3-1-RX_P: now reaches Module1.159 (USB3-1-RX_P)
- net USB3-1-RX_P: now also J6.A11 (RX2+), J6.B11 (RX1+)
- net USB3-1-D_P: now reaches Module1.163 (USB3-1-D_P)
- net USB3-1-D_P: now also J6.A6 (D+), J6.B6 (D+)
- net USB3-1-D_N: now reaches Module1.165 (USB3-1-D_N)
- net USB3-1-D_N: now also J6.A7 (D-), J6.B7 (D-)
- net USB3-1-TX_N: now reaches Module1.169 (USB3-1-TX_N)
- net USB3-1-TX_N: now also J6.A3 (TX1-), J6.B3 (TX2-)
- net USB3-1-TX_P: now reaches Module1.171 (USB3-1-TX_P)
- net USB3-1-TX_P: now also J6.A2 (TX1+), J6.B2 (TX2+)
- new net: R8.1, U7.5 (ILIM)
- new net VBUS: C25.1, C26.1, J5.A4 (VBUS), J5.A9 (VBUS), J5.B4 (VBUS), J5.B9 (VBUS), J6.A4 (VBUS), J6.A9 (VBUS), J6.B4 (VBUS), J6.B9 (VBUS), U7.6 (OUT)
- no-connect marks 5 -> 10
