File: electronics/keyboard/keyboard.kicad_pcb (KiCad board)
At the start: 2 copper layers, 87 parts, among them J0 Conn_01x04_Socket, SW0 `~, SW1 Esc, SW10 S, SW11 Z, SW12 3#, SW13 E, SW14 D, SW15 X, SW16 4$, SW17 R, SW18 F, SW19 C, SW2 Tab, SW20 5%, SW21 T, SW22 G, SW23 V, SW24 6^, SW25 Y, SW26 H, SW27 B, SW28 7&, SW29 U, SW3 Shift, SW30 J, SW31 N, SW32 8*, SW33 I, SW34 K, SW35 M, SW36 Boot, SW37 9(, SW38 O, SW39 L, SW4 1!, SW40 ,<, SW41 0), SW42 P, SW43 ;:, SW44 .>, SW45 -_, SW46 [{, SW47 '", SW48 /?, SW49 =+, SW5 Q, SW50 ]}, SW51 Enter, SW52 Space, SW53 Back, SW54 \|, SW55 Ctrl, SW56 Alt, SW57 Up, SW58 Down, SW59 Left, SW6 A, SW60 Right, SW7 FN, SW8 2@, SW9 W, U0 NCP1117-3.3_SOT223, U1 RP2040, U2 W25Q128JVS, Y0 ABM8-272-T3

Commit message: updating schematic of the keyboard
Parts:
- removed J0: Conn_01x04_Socket, Connector_Molex:Molex_PicoBlade_53048-0410_1x04_P1.25mm_Horizontal
- added J1: USB_C_Receptacle_USB2.0_16P, Connector_USB:USB_C_Receptacle_GCT_USB4085, F.Cu at (79.2, 80.6)
- added J2: Conn_01x03_MountingPin, Connector_JST:JST_SH_SM03B-SRSS-TB_1x03-1MP_P1.00mm_Horizontal, F.Cu at (77.0, 94.1)
- SW0, SW1, SW10, SW11, SW12, SW13, SW14, SW15, SW16, SW17, SW18, SW19, SW2, SW20, SW21, SW22, SW23, SW24, SW25, SW26, SW27, SW28, SW29, SW3, SW30, SW31, SW32, SW33, SW34, SW35, SW36, SW37, SW38, SW39, SW4, SW40, SW41, SW42, SW43, SW44, SW45, SW46, SW47, SW48, SW49, SW5, SW50, SW51, SW52, SW53, SW54, SW55, SW56, SW57, SW58, SW59, SW6, SW60, SW7, SW8, SW9: footprint Button_Switch_SMD:SW_SPST_PTS647_Sx70 -> Button_Switch_THT:SW_PUSH_6mm_H9.5mm
- moved R4 58.9 mm to (116.5, 81.9)
- moved C15 49.3 mm to (143.1, 86.7)
- moved R2 49.2 mm to (180.6, 94.5)
- moved C14 46.7 mm to (113.9, 79.6), turned to 90 degrees
- moved R3 45.5 mm to (178.3, 99.9)
- moved C13 44.4 mm to (117.1, 77.1), turned to 180 degrees
- moved C5 43.6 mm to (131.1, 87.6), turned to -90 degrees
- moved C3 43.6 mm to (132.6, 85.0), turned to -90 degrees
- moved R1 42.4 mm to (134.1, 85.0), turned to 90 degrees
- moved Y0 40.8 mm to (116.6, 79.4), turned to 180 degrees
- moved R0 39.6 mm to (135.6, 85.0), turned to 90 degrees
- moved U1 25.4 mm to (127.6, 81.8), turned to -90 degrees
- moved SW0 20.2 mm to (73.8, 43.3)
- moved SW1 19.6 mm to (73.8, 51.0)
- moved SW2 19.2 mm to (73.8, 58.6)
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